Commit message: Upload mesh files
Update with rendering

File: EGK/EGK 40 AIS/schunk_egk40_ais.urdf (robot description, URDF)
Before this commit: robot schunk_egk40_ais, 3 links, 2 joints
Links:
- link base_link: geometry collision mesh filename=meshes/base_link.dae; visual mesh filename=meshes/base_link.dae
